Commit message: fix arm from crashing into table

File: robotiq/robotiq_description/urdf/robotiq_85_gripper.urdf.xacro (robot description, xacro)
@@ -204,9 +204,9 @@
         </geometry>
       </visual>
-      <!-- <collision>
+      <collision>
         <geometry>
           <mesh filename="package://robotiq_description/meshes/collision/robotiq_85_finger_tip_link.stl"/>
         </geometry>
-      </collision> -->
+      </collision>
       <inertial>
         <mass value="0.019555" />
@@ -223,9 +223,9 @@
         </geometry>
       </visual>
-      <!-- <collision>
+      <collision>
         <geometry>
           <mesh filename="package://robotiq_description/meshes/collision/robotiq_85_finger_tip_link.stl"/>
         </geometry>
-      </collision> -->
+      </collision>
       <inertial>
         <mass value="0.019555" />
